File: Competition/Summer_2024/Repertoire_des_equipes/Equipe2/KiCad/V1_flappy_mouse/Section_VL.kicad_sch (KiCad schematic)
At the start: 14 parts, among them J1 ESP_DROIT, J2 ESP_GAUCHE, J3 Conn_01x08_Pin, J4 CAPACITIVE, U1 LM393

Commit message: Push pcb
Parts:
- J301: renamed from J2; footprint (none) -> Connector_PinSocket_2.54mm:PinSocket_1x22_P2.54mm_Vertical
- J302: renamed from J1; footprint (none) -> Connector_PinSocket_2.54mm:PinSocket_1x22_P2.54mm_Vertical
- J304: renamed from J3; footprint (none) -> Connector_PinSocket_2.54mm:PinSocket_1x08_P2.54mm_Vertical
- renumbered D1 to D301, D2 to D302, J4 to J303, MK1 to MK301, R5 to R301, R4 to R302, R3 to R303, R1 to R304, R2 to R305, RV1 to RV301, U1 to U301
Changed lines of the file:
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@@
 		(dnp no)
 		(fields_autoplaced yes)
-		(property "Reference" "#PWR05"
+		(property "Reference" "#PWR0307"
 			(at 99.06 83.82 0)
 			(effects
@@
 			(project "V1_flappy_mouse"
 				(path "/02a5dcc7-4b18-4a0b-b9f0-883e5dbce76c/f86b3f71-a906-482f-8366-32910134182f"
-					(reference "#PWR05")
+					(reference "#PWR0307")
 					(unit 1)
 				)
@@
 		(on_board yes)
 		(dnp no)
-		(property "Reference" "U1"
+		(property "Reference" "U301"
 			(at 88.9 129.54 0)
 			(effects
@@
 			(project "V1_flappy_mouse"
 				(path "/02a5dcc7-4b18-4a0b-b9f0-883e5dbce76c/f86b3f71-a906-482f-8366-32910134182f"
-					(reference "U1")
+					(reference "U301")
 					(unit 1)
 				)
@@
 		(dnp no)
 		(fields_autoplaced yes)
-		(property "Reference" "R3"
+		(property "Reference" "R303"
 			(at 66.04 110.49 90)
 			(effects
@@
 			(project "V1_flappy_mouse"
 				(path "/02a5dcc7-4b18-4a0b-b9f0-883e5dbce76c/f86b3f71-a906-482f-8366-32910134182f"
-					(reference "R3")
+					(reference "R303")
 					(unit 1)
 				)
@@
 		(dnp no)
 		(fields_autoplaced yes)
-		(property "Reference" "R2"
+		(property "Reference" "R305"
 			(at 129.54 105.4099 0)
 			(effects
@@
 			(project "V1_flappy_mouse"
 				(path "/02a5dcc7-4b18-4a0b-b9f0-883e5dbce76c/f86b3f71-a906-482f-8366-32910134182f"
-					(reference "R2")
+					(reference "R305")
 					(unit 1)
 				)
@@
 		(dnp no)
 		(fields_autoplaced yes)
-		(property "Reference" "R5"
+		(property "Reference" "R301"
 			(at 60.96 105.4099 0)
 			(effects
@@
 			(project "V1_flappy_mouse"
 				(path "/02a5dcc7-4b18-4a0b-b9f0-883e5dbce76c/f86b3f71-a906-482f-8366-32910134182f"
-					(reference "R5")
+					(reference "R301")
 					(unit 1)
 				)
@@
 		(dnp no)
 		(fields_autoplaced yes)
-		(property "Reference" "RV1"
+		(property "Reference" "RV301"
 			(at 71.12 105.4099 0)
 			(effects
@@
 			(project "V1_flappy_mouse"
 				(path "/02a5dcc7-4b18-4a0b-b9f0-883e5dbce76c/f86b3f71-a906-482f-8366-32910134182f"
-					(reference "RV1")
+					(reference "RV301")
 					(unit 1)
 				)
@@
 		(dnp no)
 		(fields_autoplaced yes)
-		(property "Reference" "#PWR07"
+		(property "Reference" "#PWR0308"
 			(at 125.73 29.21 0)
 			(effects
@@
 			(project "V1_flappy_mouse"
 				(path "/02a5dcc7-4b18-4a0b-b9f0-883e5dbce76c/f86b3f71-a906-482f-8366-32910134182f"
-					(reference "#PWR07")
+					(reference "#PWR0308")
 					(unit 1)
 				)
@@
 		(dnp no)
 		(fields_autoplaced yes)
-		(property "Reference" "J4"
+		(property "Reference" "J303"
 			(at 173.355 73.66 0)
 			(effects
@@
 			(project "V1_flappy_mouse"
 				(path "/02a5dcc7-4b18-4a0b-b9f0-883e5dbce76c/f86b3f71-a906-482f-8366-32910134182f"
-					(reference "J4")
+					(reference "J303")
 					(unit 1)
 				)
@@
 		(dnp no)
 		(fields_autoplaced yes)
-		(property "Reference" "#PWR03"
+		(property "Reference" "#PWR0304"
 			(at 81.28 73.66 0)
 			(effects
@@
 			(project "V1_flappy_mouse"
 				(path "/02a5dcc7-4b18-4a0b-b9f0-883e5dbce76c/f86b3f71-a906-482f-8366-32910134182f"
-					(reference "#PWR03")
+					(reference "#PWR0304")
 					(unit 1)
 				)
@@
 		(dnp no)
 		(fields_autoplaced yes)
-		(property "Reference" "R1"
+		(property "Reference" "R304"
 			(at 115.57 105.4099 0)
 			(effects
@@
 			(project "V1_flappy_mouse"
 				(path "/02a5dcc7-4b18-4a0b-b9f0-883e5dbce76c/f86b3f71-a906-482f-8366-32910134182f"
-					(reference "R1")
+					(reference "R304")
 					(unit 1)
 				)
@@
 		(dnp no)
 		(fields_autoplaced yes)
-		(property "Reference" "#PWR08"
+		(property "Reference" "#PWR0305"
 			(at 93.98 105.41 0)
 			(effects
@@
 			(project "V1_flappy_mouse"
 				(path "/02a5dcc7-4b18-4a0b-b9f0-883e5dbce76c/f86b3f71-a906-482f-8366-32910134182f"
-					(reference "#PWR08")
+					(reference "#PWR0305")
 					(unit 1)
 				)
@@
 		(dnp no)
 		(fields_autoplaced yes)
-		(property "Reference" "D1"
+		(property "Reference" "D301"
 			(at 115.57 111.6329 90)
 			(effects
@@
 			(project "V1_flappy_mouse"
 				(path "/02a5dcc7-4b18-4a0b-b9f0-883e5dbce76c/f86b3f71-a906-482f-8366-32910134182f"
-					(reference "D1")
+					(reference "D301")
 					(unit 1)
 				)
@@
 		(dnp no)
 		(fields_autoplaced yes)
-		(property "Reference" "#PWR01"
+		(property "Reference" "#PWR0302"
 			(at 81.28 22.86 0)
 			(effects
@@
 			(project "V1_flappy_mouse"
 				(path "/02a5dcc7-4b18-4a0b-b9f0-883e5dbce76c/f86b3f71-a906-482f-8366-32910134182f"
-					(reference "#PWR01")
+					(reference "#PWR0302")
 					(unit 1)
 				)
@@
 		(dnp no)
 		(fields_autoplaced yes)
-		(property "Reference" "R4"
+		(property "Reference" "R302"
 			(at 60.96 132.0799 0)
 			(effects
@@
 			(project "V1_flappy_mouse"
 				(path "/02a5dcc7-4b18-4a0b-b9f0-883e5dbce76c/f86b3f71-a906-482f-8366-32910134182f"
-					(reference "R4")
+					(reference "R302")
 					(unit 1)
 				)
@@
 		(on_board yes)
 		(dnp no)
-		(property "Reference" "J3"
+		(property "Reference" "J304"
 			(at 193.675 30.48 0)
 			(effects
@@
 			)
 		)
-		(property "Footprint" ""
+		(property "Footprint" "Connector_PinSocket_2.54mm:PinSocket_1x08_P2.54mm_Vertical"
 			(at 194.31 43.18 0)
 			(effects
@@
 			(project "V1_flappy_mouse"
 				(path "/02a5dcc7-4b18-4a0b-b9f0-883e5dbce76c/f86b3f71-a906-482f-8366-32910134182f"
-					(reference "J3")
+					(reference "J304")
 					(unit 1)
 				)
@@
 		(dnp no)
 		(fields_autoplaced yes)
-		(property "Reference" "#PWR04"
+		(property "Reference" "#PWR0301"
 			(at 76.2 83.82 0)
 			(effects
@@
 			(project "V1_flappy_mouse"
 				(path "/02a5dcc7-4b18-4a0b-b9f0-883e5dbce76c/f86b3f71-a906-482f-8366-32910134182f"
-					(reference "#PWR04")
+					(reference "#PWR0301")
 					(unit 1)
 				)
@@
 		(dnp no)
 		(fields_autoplaced yes)
-		(property "Reference" "MK1"
+		(property "Reference" "MK301"
 			(at 53.34 119.9514 0)
 			(effects
@@
 			(project "V1_flappy_mouse"
 				(path "/02a5dcc7-4b18-4a0b-b9f0-883e5dbce76c/f86b3f71-a906-482f-8366-32910134182f"
-					(reference "MK1")
+					(reference "MK301")
 					(unit 1)
 				)
@@
 		(dnp no)
 		(fields_autoplaced yes)
-		(property "Reference" "U1"
+		(property "Reference" "U301"
 			(at 105.41 120.65 0)
 			(effects
@@
 			(project "V1_flappy_mouse"
 				(path "/02a5dcc7-4b18-4a0b-b9f0-883e5dbce76c/f86b3f71-a906-482f-8366-32910134182f"
-					(reference "U1")
+					(reference "U301")
 					(unit 2)
 				)
@@
 		(dnp no)
 		(fields_autoplaced yes)
-		(property "Reference" "D2"
+		(property "Reference" "D302"
 			(at 129.54 111.6329 90)
 			(effects
@@
 			(project "V1_flappy_mouse"
 				(path "/02a5dcc7-4b18-4a0b-b9f0-883e5dbce76c/f86b3f71-a906-482f-8366-32910134182f"
-					(reference "D2")
+					(reference "D302")
 					(unit 1)
 				)
@@
 		(on_board yes)
 		(dnp no)
-		(property "Reference" "J2"
+		(property "Reference" "J301"
 			(at 81.915 17.78 0)
 			(effects
@@
 			)
 		)
-		(property "Footprint" ""
+		(property "Footprint" "Connector_PinSocket_2.54mm:PinSocket_1x22_P2.54mm_Vertical"
 			(at 82.55 48.26 0)
 			(effects
@@
 			(project "V1_flappy_mouse"
 				(path "/02a5dcc7-4b18-4a0b-b9f0-883e5dbce76c/f86b3f71-a906-482f-8366-32910134182f"
-					(reference "J2")
+					(reference "J301")
 					(unit 1)
 				)
@@
 		(dnp no)
 		(fields_autoplaced yes)
-		(property "Reference" "#PWR02"
+		(property "Reference" "#PWR0303"
 			(at 81.28 25.4 0)
 			(effects
@@
 			(project "V1_flappy_mouse"
 				(path "/02a5dcc7-4b18-4a0b-b9f0-883e5dbce76c/f86b3f71-a906-482f-8366-32910134182f"
-					(reference "#PWR02")
+					(reference "#PWR0303")
 					(unit 1)
 				)
@@
 		(dnp no)
 		(fields_autoplaced yes)
-		(property "Reference" "J1"
+		(property "Reference" "J302"
 			(at 93.345 17.78 0)
 			(effects
@@
 			)
 		)
-		(property "Footprint" ""
+		(property "Footprint" "Connector_PinSocket_2.54mm:PinSocket_1x22_P2.54mm_Vertical"
 			(at 92.71 48.26 0)
 			(effects
@@
 			(project "V1_flappy_mouse"
 				(path "/02a5dcc7-4b18-4a0b-b9f0-883e5dbce76c/f86b3f71-a906-482f-8366-32910134182f"
-					(reference "J1")
+					(reference "J302")
 					(unit 1)
 				)
@@
 		(dnp no)
 		(fields_autoplaced yes)
-		(property "Reference" "#PWR06"
+		(property "Reference" "#PWR0306"
 			(at 93.98 147.32 0)
 			(effects
@@
 			(project "V1_flappy_mouse"
 				(path "/02a5dcc7-4b18-4a0b-b9f0-883e5dbce76c/f86b3f71-a906-482f-8366-32910134182f"
-					(reference "#PWR06")
-					(unit 1)
-				)
+					(reference "#PWR0306")
+					(unit 1)
+				)

Commit message: Taking a break, i will come back later today
Parts:
- removed J303: CAPACITIVE, symbol Connector:Conn_01x04_Pin
- added JP1: SolderJumper_AOUT, symbol Jumper:SolderJumper_2_Open
- added JP2: SolderJumper_DOUT, symbol Jumper:SolderJumper_2_Open
- added R306: 10K, symbol Device:R
- added TP5: Touchpad_click_gauche, Librairie_touchpad:Touchpad_biz_rect, symbol Connector:TestPoint_Alt
- added TP6: Touchpad_scroll4, Librairie_touchpad:Touchpad_biz_rect, symbol Connector:TestPoint_Alt
- added TP7: Touchpad_scroll5, Librairie_touchpad:Touchpad_biz_rect, symbol Connector:TestPoint_Alt
- added TP8: Touchpad_scroll6, Librairie_touchpad:Touchpad_biz_rect, symbol Connector:TestPoint_Alt
- J304: value Conn_01x08_Pin -> Conn_TFT_display
Connections:
- net AOUT is gone; now on an unnamed net: R303.2, RV301.1, U301.2 (-)
- net +3.3V: now also R306.1
- net TOUCH4/GPIO4: now also TP5.1
- net TOUCH5/GPIO5: now also TP6.1
- net TOUCH6/GPIO6: now also TP7.1
- net TOUCH7/GPIO7: now also TP8.1
- net U1RXD/GPIO18: now also JP1.2 (B)
- net U1TXD/GPIO17: now also JP2.2 (B)
- net at RV301.2: now also JP1.1 (A)
- net DOUT: no longer names the net of U301.1, U301.6 (-)
- net DOUT: now also JP2.1 (A), R306.2
Other:
- removed sheet CAPACITIVE_TOUCH
- removed sheet ESP32_Pin_out
- removed sheet SOUND_SENSOR
- removed sheet TFT_DISPLAY
- note added: "8 COUPS D'ENCODEUR MAX PAR SCROLL POUR LA SCROLL WHEEL"
- note added: "AOUT"
- note added: "CAPACITIVE TOUCH"
- note added: "DOUT"
- note added: "ESP32-S3 PINOUT"
- note added: "SOUND SENSOR"
- note added: "TFT DISPLAY"
- note added: "VÉRIFIER SI JE NE PEUX CHANGER LE GPIO36/FSPICLK POUR QQCH D'AUTRE OU CELUI DE JACOB"
- note added: "VÉRIFIER SI Y'AURAIT PAS MOYEN DE TUNER MON CIRCUIT POUR"
- note removed: "JE PENSAIS CONNECTER DES PADS DE MÉTAL JE SAIS PAS CE QUE TU EN PENSES"
- moved on the sheet: J304, MK301, R301, R302
