File: Competition/Summer_2024/Repertoire_des_equipes/Equipe2/KiCad/V1_flappy_mouse/Section_JT.kicad_sch (KiCad schematic)
At the start: 0 parts

Commit message: Push des changements fait
Parts:
- added J201: Conn_accelerometer_I2C, symbol Connector_Generic:Conn_01x07
- added J202: Conn_01x05_no_connect(SPI), symbol Connector_Generic:Conn_01x05
- added J203: Conn_Module_SD, symbol Connector_Generic:Conn_01x06
- added SW201: JS102011JAQN, Button_Switch_SMD:SW_SPDT_CK-JS102011SAQN, symbol Switch:SW_SPDT
- added TP201: Touchpad_click_droit, TestPoint:TestPoint_Pad_D4.0mm, symbol Connector:TestPoint_Alt
- added TP202: Touchpad_scroll1, TestPoint:TestPoint_Pad_D4.0mm, symbol Connector:TestPoint_Alt
- added TP203: Touchpad_scroll2, TestPoint:TestPoint_Pad_D4.0mm, symbol Connector:TestPoint_Alt
- added TP204: Touchpad_scroll3, TestPoint:TestPoint_Pad_D4.0mm, symbol Connector:TestPoint_Alt
Connections:
- new net +3.3V: J201.1 (Pin_1), J201.2 (Pin_2), J203.1 (Pin_1), SW201.1 (A)
- new net FSPICS0/TOUCH10/GPIO10: TP203.1
- new net FSPID/TOUCH11/GPIO11: TP204.1
- new net FSPIHD/TOUCH9/GPIO9: TP202.1
- new net GND: J201.3 (Pin_3), J201.7 (Pin_7), J203.6 (Pin_6), SW201.3 (C)
- new net GPIO2/TOUCH2/ADC1_1/SCL1: J201.4 (Pin_4)
- new net GPIO35/FSPID: J203.3 (Pin_3)
- new net GPIO36/FSPICLK: J203.4 (Pin_4)
- new net GPIO37/FSPIQ: J203.5 (Pin_5)
- new net JTAG/TOUCH3/SDA1/GPIO3: J201.5 (Pin_5)
- new net TOUCH8/GPIO8: TP201.1
- new net U0CTS/GPIO16: J203.2 (Pin_2)
- new net U0RTS/GPIO15: SW201.2 (B)
- no-connect marks 0 -> 6
Other:
- note added: "Accéléromètre en I2C BMI160 Adresse I2C: 0x68"
- note added: "CS"
- note added: "Connecteur pour lecteur de carte µSD. CS: GPIO16"
- note added: "MOSI CLK MISO"
- note added: "Switch permettant de toggle entre différents mode de fonctionnement"
- note added: "Touchpad de Jacob pour le côté droit du PCB"

Commit message: Push pcb
Parts:
- J201: renamed from J202; footprint (none) -> Connector_PinSocket_2.54mm:PinSocket_1x05_P2.54mm_Vertical
- J202: renamed from J201; footprint (none) -> Connector_PinSocket_2.54mm:PinSocket_1x07_P2.54mm_Vertical
- J203: footprint (none) -> Connector_PinSocket_2.54mm:PinSocket_1x06_P2.54mm_Vertical
- SW201: footprint Button_Switch_SMD:SW_SPDT_CK-JS102011SAQN -> Button_Switch_SMD:SW_SPDT_CK_JS102011SAQN
- TP201: footprint TestPoint:TestPoint_Pad_D4.0mm -> Librairie_touchpad:Touchpad_biz_rect
- TP202, TP203, TP204: footprint TestPoint:TestPoint_Pad_D4.0mm -> Librairie_touchpad:Touchpad_slider
Changed lines of the file:
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@@
 		(dnp no)
 		(fields_autoplaced yes)
-		(property "Reference" "#PWR0202"
+		(property "Reference" "#PWR0203"
 			(at 52.07 36.83 0)
 			(effects
@@
 			(project "V1_flappy_mouse"
 				(path "/02a5dcc7-4b18-4a0b-b9f0-883e5dbce76c/c9bdbe16-fb84-44c9-b5f6-cb197b4bed59"
-					(reference "#PWR0202")
+					(reference "#PWR0203")
 					(unit 1)
 				)
@@
 			)
 		)
-		(property "Footprint" ""
+		(property "Footprint" "Connector_PinSocket_2.54mm:PinSocket_1x06_P2.54mm_Vertical"
 			(at 83.82 49.53 0)
 			(effects
@@
 			)
 		)
-		(property "Footprint" "TestPoint:TestPoint_Pad_D4.0mm"
+		(property "Footprint" "Librairie_touchpad:Touchpad_slider"
 			(at 146.05 21.59 0)
 			(effects
@@
 			)
 		)
-		(property "Footprint" "TestPoint:TestPoint_Pad_D4.0mm"
+		(property "Footprint" "Librairie_touchpad:Touchpad_slider"
 			(at 167.64 21.59 0)
 			(effects
@@
 		(dnp no)
 		(fields_autoplaced yes)
-		(property "Reference" "#PWR0201"
+		(property "Reference" "#PWR0205"
 			(at 82.55 15.24 0)
 			(effects
@@
 			(project "V1_flappy_mouse"
 				(path "/02a5dcc7-4b18-4a0b-b9f0-883e5dbce76c/c9bdbe16-fb84-44c9-b5f6-cb197b4bed59"
-					(reference "#PWR0201")
+					(reference "#PWR0205")
 					(unit 1)
 				)
@@
 		(on_board yes)
 		(dnp no)
-		(property "Reference" "#PWR0204"
+		(property "Reference" "#PWR0201"
 			(at 24.13 60.96 0)
 			(effects
@@
 			(project "V1_flappy_mouse"
 				(path "/02a5dcc7-4b18-4a0b-b9f0-883e5dbce76c/c9bdbe16-fb84-44c9-b5f6-cb197b4bed59"
-					(reference "#PWR0204")
+					(reference "#PWR0201")
 					(unit 1)
 				)
@@
 		(dnp no)
 		(fields_autoplaced yes)
-		(property "Reference" "#PWR0203"
+		(property "Reference" "#PWR0206"
 			(at 82.55 17.78 0)
 			(effects
@@
 			(project "V1_flappy_mouse"
 				(path "/02a5dcc7-4b18-4a0b-b9f0-883e5dbce76c/c9bdbe16-fb84-44c9-b5f6-cb197b4bed59"
-					(reference "#PWR0203")
+					(reference "#PWR0206")
 					(unit 1)
 				)
@@
 			)
 		)
-		(property "Footprint" "TestPoint:TestPoint_Pad_D4.0mm"
+		(property "Footprint" "Librairie_touchpad:Touchpad_slider"
 			(at 189.23 21.59 0)
 			(effects
@@
 		(on_board yes)
 		(dnp no)
-		(property "Reference" "J201"
+		(property "Reference" "J202"
 			(at 81.28 32.766 0)
 			(effects
@@
 			)
 		)
-		(property "Footprint" ""
+		(property "Footprint" "Connector_PinSocket_2.54mm:PinSocket_1x07_P2.54mm_Vertical"
 			(at 83.82 22.86 0)
 			(effects
@@
 			(project "V1_flappy_mouse"
 				(path "/02a5dcc7-4b18-4a0b-b9f0-883e5dbce76c/c9bdbe16-fb84-44c9-b5f6-cb197b4bed59"
-					(reference "J201")
+					(reference "J202")
 					(unit 1)
 				)
@@
 		(dnp no)
 		(fields_autoplaced yes)
-		(property "Reference" "#PWR0206"
+		(property "Reference" "#PWR0207"
 			(at 82.55 44.45 0)
 			(effects
@@
 			(project "V1_flappy_mouse"
 				(path "/02a5dcc7-4b18-4a0b-b9f0-883e5dbce76c/c9bdbe16-fb84-44c9-b5f6-cb197b4bed59"
-					(reference "#PWR0206")
+					(reference "#PWR0207")
 					(unit 1)
 				)
@@
 			)
 		)
-		(property "Footprint" "TestPoint:TestPoint_Pad_D4.0mm"
+		(property "Footprint" "Librairie_touchpad:Touchpad_biz_rect"
 			(at 121.92 21.59 0)
 			(effects
@@
 			)
 		)
-		(property "Footprint" "Button_Switch_SMD:SW_SPDT_CK-JS102011SAQN"
+		(property "Footprint" "Button_Switch_SMD:SW_SPDT_CK_JS102011SAQN"
 			(at 30.48 48.26 0)
 			(effects
@@
 		(dnp no)
 		(fields_autoplaced yes)
-		(property "Reference" "#PWR0205"
+		(property "Reference" "#PWR0202"
 			(at 29.21 45.72 0)
 			(effects
@@
 			(project "V1_flappy_mouse"
 				(path "/02a5dcc7-4b18-4a0b-b9f0-883e5dbce76c/c9bdbe16-fb84-44c9-b5f6-cb197b4bed59"
-					(reference "#PWR0205")
+					(reference "#PWR0202")
 					(unit 1)
 				)
@@
 		(dnp no)
 		(fields_autoplaced yes)
-		(property "Reference" "J202"
+		(property "Reference" "J201"
 			(at 21.59 19.0499 0)
 			(effects
@@
 			)
 		)
-		(property "Footprint" ""
+		(property "Footprint" "Connector_PinSocket_2.54mm:PinSocket_1x05_P2.54mm_Vertical"
 			(at 19.05 20.32 0)
 			(effects
@@
 			(project "V1_flappy_mouse"
 				(path "/02a5dcc7-4b18-4a0b-b9f0-883e5dbce76c/c9bdbe16-fb84-44c9-b5f6-cb197b4bed59"
-					(reference "J202")
+					(reference "J201")
 					(unit 1)
 				)
@@
 		(on_board yes)
 		(dnp no)
-		(property "Reference" "#PWR0207"
+		(property "Reference" "#PWR0204"
 			(at 77.47 67.31 0)
 			(effects
@@
 			(project "V1_flappy_mouse"
 				(path "/02a5dcc7-4b18-4a0b-b9f0-883e5dbce76c/c9bdbe16-fb84-44c9-b5f6-cb197b4bed59"
-					(reference "#PWR0207")
-					(unit 1)
-				)
+					(reference "#PWR0204")
+					(unit 1)
+				)
