File: Documentation/1_Plans_elect/Schema/Schema.kicad_pcb (KiCad board)
At the start: 2 copper layers, 0.6 x 11.1 mm, 23 parts, among them J1 Conn_01x22, J2 Conn_01x22, J3 Conn_01x10, J4 Conn_01x14, SW1 RotaryEncoder_Switch, SW2 RotaryEncoder_Switch, SW3 RotaryEncoder

Commit message: quick fix
Parts:
- moved SW3 5.16 mm to (181.6, 83.5), turned to 0 degrees
Connections:
- SW3 pad 1: (no net) -> GND
- SW3 pad 2: (no net) -> Net-(C6-Pad1)
- SW3 pad 3: (no net) -> Net-(C5-Pad1)
Other:
- board size 0.6 x 11.1 mm -> 11 x 0.6 mm
Changed lines of the file:
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@@
 		)
 		(property ki_fp_filters "R_*")
-		(sheetname "Root")
+		(sheetname "Racine")
 		(sheetfile "Schema.kicad_sch")
 		(attr smd)
@@
 		)
 		(property ki_fp_filters "R_*")
-		(sheetname "Root")
+		(sheetname "Racine")
 		(sheetfile "Schema.kicad_sch")
 		(attr smd)
@@
 		)
 		(property ki_fp_filters "R_*")
-		(sheetname "Root")
+		(sheetname "Racine")
 		(sheetfile "Schema.kicad_sch")
 		(attr smd)
@@
 		)
 		(property ki_fp_filters "C_*")
-		(sheetname "Root")
+		(sheetname "Racine")
 		(sheetfile "Schema.kicad_sch")
 		(attr smd)
@@
 		)
 		(property ki_fp_filters "Connector*:*_1x??_*")
-		(sheetname "Root")
+		(sheetname "Racine")
 		(sheetfile "Schema.kicad_sch")
 		(attr through_hole)
@@
 		)
 		(property ki_fp_filters "Connector*:*_1x??_*")
-		(sheetname "Root")
+		(sheetname "Racine")
 		(sheetfile "Schema.kicad_sch")
 		(attr through_hole)
@@
 		)
 		(fp_text user "${REFERENCE}"
-			(at 0 6.5 360)
+			(at 0 6.5 0)
 			(layer "F.Fab")
 			(effects
@@
 		)
 		(property ki_fp_filters "R_*")
-		(sheetname "Root")
+		(sheetname "Racine")
 		(sheetfile "Schema.kicad_sch")
 		(attr smd)
@@
 		)
 		(property ki_fp_filters "R_*")
-		(sheetname "Root")
+		(sheetname "Racine")
 		(sheetfile "Schema.kicad_sch")
 		(attr smd)
@@
 		)
 		(property ki_fp_filters "R_*")
-		(sheetname "Root")
+		(sheetname "Racine")
 		(sheetfile "Schema.kicad_sch")
 		(attr smd)
@@
 		)
 		(property ki_fp_filters "Connector*:*_1x??_*")
-		(sheetname "Root")
+		(sheetname "Racine")
 		(sheetfile "Schema.kicad_sch")
 		(attr through_hole)
@@
 		)
 		(fp_text user "${REFERENCE}"
-			(at 0 10.5 360)
+			(at 0 10.5 0)
 			(layer "F.Fab")
 			(effects
@@
 		)
 		(property ki_fp_filters "C_*")
-		(sheetname "Root")
+		(sheetname "Racine")
 		(sheetfile "Schema.kicad_sch")
 		(attr smd)
@@
 		)
 		(property ki_fp_filters "R_*")
-		(sheetname "Root")
+		(sheetname "Racine")
 		(sheetfile "Schema.kicad_sch")
 		(attr smd)
@@
 		)
 		(property ki_fp_filters "RotaryEncoder*Switch*")
-		(sheetname "Root")
+		(sheetname "Racine")
 		(sheetfile "Schema.kicad_sch")
 		(attr through_hole)
@@
 		)
 		(property ki_fp_filters "C_*")
-		(sheetname "Root")
+		(sheetname "Racine")
 		(sheetfile "Schema.kicad_sch")
 		(attr smd)
@@
 		)
 		(property ki_fp_filters "R_*")
-		(sheetname "Root")
+		(sheetname "Racine")
 		(sheetfile "Schema.kicad_sch")
 		(attr smd)
@@
 		)
 		(property ki_fp_filters "C_*")
-		(sheetname "Root")
+		(sheetname "Racine")
 		(sheetfile "Schema.kicad_sch")
 		(attr smd)
@@
 		)
 		(property ki_fp_filters "C_*")
-		(sheetname "Root")
+		(sheetname "Racine")
 		(sheetfile "Schema.kicad_sch")
 		(attr smd)
@@
 		)
 		(property ki_fp_filters "Connector*:*_1x??_*")
-		(sheetname "Root")
+		(sheetname "Racine")
 		(sheetfile "Schema.kicad_sch")
 		(attr through_hole)
@@
 		)
 		(fp_text user "${REFERENCE}"
-			(at 0 10.5 360)
+			(at 0 10.5 0)
 			(layer "F.Fab")
 			(effects
@@
 		)
 		(property ki_fp_filters "C_*")
-		(sheetname "Root")
+		(sheetname "Racine")
 		(sheetfile "Schema.kicad_sch")
 		(attr smd)
@@
 		)
 		(property ki_fp_filters "R_*")
-		(sheetname "Root")
+		(sheetname "Racine")
 		(sheetfile "Schema.kicad_sch")
 		(attr smd)
@@
 	(footprint "footprints:EN10HT_BIT"
 		(layer "F.Cu")
-		(at 186.4909 82 -90)
+		(at 181.55 83.5)
 		(tags "EN10HT1212N5HH3 ")
 		(property "Reference" "SW3"
-			(at 2.5 0 -90)
+			(at 2.5 0 0)
 			(unlocked yes)
 			(layer "F.SilkS")
@@
 		)
 		(property "Value" "RotaryEncoder"
-			(at 2.5 0 -90)
+			(at 2.5 0 0)
 			(unlocked yes)
 			(layer "F.Fab")
@@
 		)
 		(property "Footprint" "footprints:EN10HT_BIT"
-			(at 0 0 90)
+			(at 0 0 0)
+			(unlocked yes)
 			(layer "F.Fab")
 			(hide yes)
@@
 				(font
 					(size 1.27 1.27)
-					(thickness 0.15)
 				)
 			)
 		)
 		(property "Datasheet" ""
-			(at 0 0 90)
+			(at 0 0 0)
+			(unlocked yes)
 			(layer "F.Fab")
 			(hide yes)
@@
 				(font
 					(size 1.27 1.27)
-					(thickness 0.15)
 				)
 			)
 		)
 		(property "Description" "Rotary encoder, dual channel, incremental quadrate outputs"
-			(at 0 0 90)
+			(at 0 0 0)
+			(unlocked yes)
 			(layer "F.Fab")
 			(hide yes)
@@
 				(font
 					(size 1.27 1.27)
-					(thickness 0.15)
 				)
 			)
 		)
 		(property ki_fp_filters "RotaryEncoder*")
-		(sheetname "Root")
+		(sheetname "Racine")
 		(sheetfile "Schema.kicad_sch")
 		(attr through_hole)
@@
 		)
 		(fp_line
-			(start -2.8213 10.3186)
-			(end 7.8213 10.3186)
+			(start -2.8213 1.073)
+			(end -2.8213 3.605561)
 			(stroke
 				(width 0.1524)
@@
 		)
 		(fp_line
-			(start 7.8213 10.3186)
-			(end 7.8213 7.394437)
+			(start -2.8213 7.394437)
+			(end -2.8213 10.3186)
 			(stroke
 				(width 0.1524)
@@
 		)
 		(fp_line
-			(start -2.8213 7.394437)
-			(end -2.8213 10.3186)
+			(start -2.8213 10.3186)
+			(end 7.8213 10.3186)
 			(stroke
 				(width 0.1524)
@@
 		)
 		(fp_line
-			(start 7.8213 3.605561)
-			(end 7.8213 1.073)
+			(start -0.499675 1.073)
+			(end -2.8213 1.073)
 			(stroke
 				(width 0.1524)
@@
 		)
 		(fp_line
-			(start -2.8213 1.073)
-			(end -2.8213 3.605561)
+			(start 2.000325 1.073)
+			(end 0.499675 1.073)
 			(stroke
 				(width 0.1524)
@@
 		)
 		(fp_line
-			(start -0.499675 1.073)
-			(end -2.8213 1.073)
+			(start 4.500325 1.073)
+			(end 2.999675 1.073)
 			(stroke
 				(width 0.1524)
@@
 		)
 		(fp_line
-			(start 2.000325 1.073)
-			(end 0.499675 1.073)
+			(start 7.8213 1.073)
+			(end 5.499675 1.073)
 			(stroke
 				(width 0.1524)
@@
 		)
 		(fp_line
-			(start 4.500325 1.073)
-			(end 2.999675 1.073)
+			(start 7.8213 3.605561)
+			(end 7.8213 1.073)
 			(stroke
 				(width 0.1524)
@@
 		)
 		(fp_line
-			(start 7.8213 1.073)
-			(end 5.499675 1.073)
+			(start 7.8213 10.3186)
+			(end 7.8213 7.394437)
 			(stroke
 				(width 0.1524)
@@
 		)
 		(fp_line
-			(start -4.536301 10.4456)
-			(end 9.536301 10.4456)
+			(start -4.536301 -1.1049)
+			(end -4.536301 10.4456)
 			(stroke
 				(width 0.1524)
@@
 		)
 		(fp_line
-			(start 9.536301 10.4456)
-			(end 9.536301 -1.1049)
+			(start -4.536301 10.4456)
+			(end 9.536301 10.4456)
 			(stroke
 				(width 0.1524)
@@
 		)
 		(fp_line
-			(start -4.536301 -1.1049)
-			(end -4.536301 10.4456)
+			(start 9.536301 -1.1049)
+			(end -4.536301 -1.1049)
 			(stroke
 				(width 0.1524)
@@
 		)
 		(fp_line
-			(start 9.536301 -1.1049)
-			(end -4.536301 -1.1049)
+			(start 9.536301 10.4456)
+			(end 9.536301 -1.1049)
 			(stroke
 				(width 0.1524)
@@
 		)
 		(fp_line
-			(start -2.6943 10.1916)
-			(end 7.6943 10.1916)
+			(start -2.6943 1.2)
+			(end -2.6943 10.1916)
 			(stroke
 				(width 0.0254)
@@
 		)
 		(fp_line
-			(start 7.6943 10.1916)
-			(end 7.6943 1.2)
+			(start -2.6943 10.1916)
+			(end 7.6943 10.1916)
 			(stroke
 				(width 0.0254)
@@
 		)
 		(fp_line
-			(start -2.6943 1.2)
-			(end -2.6943 10.1916)
+			(start 7.6943 1.2)
+			(end -2.6943 1.2)
 			(stroke
 				(width 0.0254)
@@
 		)
 		(fp_line
-			(start 7.6943 1.2)
-			(end -2.6943 1.2)
+			(start 7.6943 10.1916)
+			(end 7.6943 1.2)
 			(stroke
 				(width 0.0254)
@@
 		)
 		(fp_text user "${REFERENCE}"
-			(at 2.5 0 -90)
+			(at 2.5 0 0)
 			(unlocked yes)
 			(layer "F.Fab")
@@
 		)
 		(pad "" np_thru_hole circle
-			(at -3.025 5.182499 270)
+			(at -3.025 5.182499)
 			(size 2.0066 2.0066)
 			(drill 2.0066)
@@
 		)
 		(pad "" np_thru_hole circle
-			(at -3.025 5.817499 270)
+			(at -3.025 5.817499)
 			(size 2.0066 2.0066)
 			(drill 2.0066)
@@
 		)
 		(pad "" np_thru_hole circle
-			(at 8.025 5.182499 270)
+			(at 8.025 5.182499)
 			(size 2.0066 2.0066)
 			(drill 2.0066)
@@
 		)
 		(pad "" np_thru_hole circle
-			(at 8.025 5.817499 270)
+			(at 8.025 5.817499)
 			(size 2.0066 2.0066)
 			(drill 2.0066)
@@
 		)
 		(pad "1" thru_hole circle
-			(at 0 0 270)
+			(at 0 0)
 			(size 1.7018 1.7018)
 			(drill 1.1938)
 			(layers "*.Cu" "*.Mask")
 			(remove_unused_layers no)
+			(net 2 "GND")
+			(pinfunction "1")
+			(pintype "passive")
 		)
 		(pad "2" thru_hole circle
-			(at 2.5 0 270)
+			(at 2.5 0)
 			(size 1.7018 1.7018)
 			(drill 1.1938)
 			(layers "*.Cu" "*.Mask")
 			(remove_unused_layers no)
+			(net 4 "Net-(C6-Pad1)")
+			(pinfunction "2")
+			(pintype "passive")
 		)
 		(pad "3" thru_hole circle
-			(at 5 0 270)
+			(at 5 0)
 			(size 1.7018 1.7018)
 			(drill 1.1938)
 			(layers "*.Cu" "*.Mask")
 			(remove_unused_layers no)
+			(net 3 "Net-(C5-Pad1)")
+			(pinfunction "3")
+			(pintype "passive")
 		)
 		(pad "4" smd oval
-			(at -3.025 5.499999 270)
+			(at -3.025 5.499999)
 			(size 2.5146 3.1496)
 			(layers "F.Cu" "F.Paste" "F.Mask")
 		)
 		(pad "5" smd oval
-			(at 8.025 5.499999 270)
+			(at 8.025 5.499999)
 			(size 2.5146 3.1496)
 			(layers "F.Cu" "F.Paste" "F.Mask")
@@
 		)
 		(property ki_fp_filters "RotaryEncoder*Switch*")
-		(sheetname "Root")
+		(sheetname "Racine")
 		(sheetfile "Schema.kicad_sch")
 		(attr through_hole)
@@
 		)
 		(property ki_fp_filters "R_*")
-		(sheetname "Root")
+		(sheetname "Racine")
 		(sheetfile "Schema.kicad_sch")
 		(attr smd)
