File: Documentation/1_Plans_elect/Schema/Schema.kicad_sch (KiCad schematic)
At the start: 25 parts, among them J1 Conn_01x22, J2 Conn_01x22, J3 Conn_01x10, SW1 RotaryEncoder, SW2 RotaryEncoder, SW3 RotaryEncoder

Commit message: tit modif
Parts:
- added J4: Conn_01x14, symbol Connector_Generic:Conn_01x14
Connections:
- net 5Vin is gone; now on net 5V: J1.21 (Pin_21)
- net GND: now also J4.2 (Pin_2)
- net VCC: now also J4.1 (Pin_1)
- new net CS: J4.3 (Pin_3)
- new net DC: J4.5 (Pin_5)
- new net LED: J4.8 (Pin_8)
- new net RESET: J4.4 (Pin_4)
- new net SCK: J4.7 (Pin_7)
- new net SDI: J4.6 (Pin_6)
- new net SDO: J4.9 (Pin_9)
- new net T_CLK: J4.10 (Pin_10)
- new net T_CS: J4.11 (Pin_11)
- new net T_DIN: J4.12 (Pin_12)
- new net T_DO: J4.13 (Pin_13)
- new net T_IRQ: J4.14 (Pin_14)

Commit message: PCB
J'ai un bug ou les footprint ne s'associe pas correctement
Parts:
- removed C3, C4: 22nF, symbol Device:C
- removed C7: C, symbol Device:C
- removed R5, R6, R7, R8: 10K, symbol Device:R
- removed SW1, SW2: RotaryEncoder, symbol Device:RotaryEncoder
- added C11, C8: 100nF, Capacitor_SMD:C_0805_2012Metric_Pad1.18x1.45mm_HandSolder, symbol Device:C
- added R13, R16: 1K, Resistor_SMD:R_0805_2012Metric_Pad1.20x1.40mm_HandSolder, symbol Device:R
- added SW1, SW2: RotaryEncoder_Switch, Rotary_Encoder:RotaryEncoder_Alps_EC11E-Switch_Vertical_H20mm, symbol Device:RotaryEncoder_Switch
- C1, C2: value 22nF -> 100nF; footprint (none) -> Capacitor_SMD:C_0805_2012Metric_Pad1.18x1.45mm_HandSolder
- C5, C6: footprint (none) -> Capacitor_SMD:C_0805_2012Metric_Pad1.18x1.45mm_HandSolder
- J1, J2: footprint (none) -> Connector_PinHeader_1.00mm:PinHeader_1x22_P1.00mm_Vertical
- J3: footprint (none) -> Connector_PinHeader_1.00mm:PinHeader_1x10_P1.00mm_Vertical
- J4: footprint (none) -> Connector_PinHeader_1.00mm:PinHeader_1x14_P1.00mm_Vertical
- R1, R2, R3, R4: value 10K -> 1K; footprint (none) -> Resistor_SMD:R_0805_2012Metric_Pad1.20x1.40mm_HandSolder
- R10, R11, R12, R9: footprint (none) -> Resistor_SMD:R_0805_2012Metric_Pad1.20x1.40mm_HandSolder
- SW3: footprint (none) -> footprints:EN10HT_BIT
Connections:
- net ADO is gone; now on net GND: J3.4 (Pin_4)
- net CS is gone; now on net GPIO14-CS: J4.3 (Pin_3)
- net DC is gone; now on net GPIO12-DC: J4.5 (Pin_5)
- net LED is gone; now on net 3V3: J4.8 (Pin_8)
- net RESET is gone; now on net GPIO13-RESET: J4.4 (Pin_4)
- net SCK is gone; now on net GPIO10-SCk: J4.7 (Pin_7)
- net SCL is gone; now on net GPIO1-SCL: J3.8 (Pin_8)
- net SDA is gone; now on net GPIO2-SDA: J3.7 (Pin_7)
- net SDI is gone; now on net GPIO11-SDI: J4.6 (Pin_6)
- net SDO is gone; now on net GPIO9-SDO: J4.9 (Pin_9)
- net VCC is gone; now on net 3V3: J3.10 (Pin_10), J4.1 (Pin_1)
- net chA-S is gone; now on net GPIO38_chA_S: R11.1
- net chA-X is gone; now on net 3V3: R4.1
- net chB-S is gone; now on net GPIO37-chB_S: R9.2
- net chB-X is gone; now on net GPIO42-chA_X: R1.2
- net 3V3: now also C1.1, C2.1, R1.1, R10.1, R12.1, R2.1, C11.1, C8.1, R13.1
- net 5V: no longer R10.1, R12.1, R2.1, R3.1
- net GND: now also SW3.A, C11.2, C8.2, SW1.C, SW1.S1, SW2.C, SW2.S1; no longer SW3.C
- net at C5.1, R10.2, R9.1: now also SW3.B; no longer SW3.A
- net at C6.1, R11.2, R12.2: now also SW3.C; no longer SW3.B
- net 0 renamed GPIO0
- net 1 renamed GPIO1-SCL
- net 10 renamed GPIO10-SCk
- net 11 renamed GPIO11-SDI
- net 12 renamed GPIO12-DC
- net 13 renamed GPIO13-RESET
- net 14 renamed GPIO14-CS
- net 15 renamed GPIO15
- net 16 renamed GPIO16
- net 17 renamed GPIO17
- net 18 renamed GPIO18
- net 19 renamed GPIO19
- net 2 renamed GPIO2-SDA
- net 20 renamed GPIO20
- net 21 renamed GPIO21-BSW3
- net 3 renamed GPIO3
- net 35 renamed GPIO35
- net 36 renamed GPIO36
- net 37 renamed GPIO37-chB_S
- net 38 renamed GPIO38_chA_S
- net 39 renamed GPIO39-chB_Y
- net GPIO39-chB_Y: now also R13.2, SW2.B
- net 4 renamed GPIO4
- net 40 renamed GPIO40-chA_Y
- net GPIO40-chA_Y: now also R4.2, SW2.A
- net 41 renamed GPIO41-chB_X
- net GPIO41-chB_X: now also R2.2, SW1.B
- net 42 renamed GPIO42-chA_X
- net GPIO42-chA_X: now also SW1.A
- net 45 renamed GPIO45
- net 46 renamed GPIO46
- net 47 renamed GPIO47-BSW2
- net GPIO47-BSW2: now also R16.1
- net 48 renamed GPIO48-BSW1
- net GPIO48-BSW1: now also R3.2
- net 5 renamed GPIO5
- net 6 renamed GPIO6
- net 7 renamed GPIO7
- net 8 renamed GPIO8
- net 9 renamed GPIO9-SDO
- new net: R3.1, SW1.S2
- new net: R16.2, SW2.S2
Other:
- note added: "3V3"
- note added: "CS"
- note added: "DC"
- note added: "GND"
- note added: "LED"
- note added: "Not used"
- note added: "RESET"
- note added: "SCK"
- note added: "SDI"
- note added: "SDO"
- note added: "VCC"
- moved on the sheet: C1, C2, C5, C6, R10, R11, R12, R9

Commit message: quick fix
Connections:
- net GND: now also SW3.1; no longer SW3.A
- net at C5.1, R10.2, R9.1: now also SW3.3; no longer SW3.B
- net at C6.1, R11.2, R12.2: now also SW3.2; no longer SW3.C
Changed lines of the file:
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@@
 		)
 		(instances
-			(project ""
+			(project "Schema"
 				(path "/3d35b564-5845-42c9-844e-b1ab721a1005"
 					(reference "J1")
@@
 		)
 		(instances
-			(project ""
+			(project "Schema"
 				(path "/3d35b564-5845-42c9-844e-b1ab721a1005"
 					(reference "SW1")
@@
 			)
 		)
-		(pin "A"
-		)
-		(pin "C"
-		)
-		(pin "B"
-		)
-		(instances
-			(project ""
+		(pin "2"
+		)
+		(pin "1"
+		)
+		(pin "3"
+		)
+		(instances
+			(project "Schema"
 				(path "/3d35b564-5845-42c9-844e-b1ab721a1005"
 					(reference "SW3")
@@
 		)
 		(instances
-			(project ""
+			(project "Schema"
 				(path "/3d35b564-5845-42c9-844e-b1ab721a1005"
 					(reference "J2")
@@
 		)
 		(instances
-			(project ""
+			(project "Schema"
 				(path "/3d35b564-5845-42c9-844e-b1ab721a1005"
 					(reference "R3")
@@
 		)
 		(instances
-			(project ""
+			(project "Schema"
 				(path "/3d35b564-5845-42c9-844e-b1ab721a1005"
 					(reference "J4")
@@
 		)
 		(instances
-			(project ""
+			(project "Schema"
 				(path "/3d35b564-5845-42c9-844e-b1ab721a1005"
 					(reference "#PWR01")
@@
 		)
 		(instances
-			(project ""
+			(project "Schema"
 				(path "/3d35b564-5845-42c9-844e-b1ab721a1005"
 					(reference "SW2")
@@
 		)
 		(instances
-			(project ""
+			(project "Schema"
 				(path "/3d35b564-5845-42c9-844e-b1ab721a1005"
 					(reference "C1")
@@
 		)
 		(instances
-			(project ""
+			(project "Schema"
 				(path "/3d35b564-5845-42c9-844e-b1ab721a1005"
 					(reference "J3")
