File: Competition/Summer_2024/Document_of_comp/Medal_V1/Ruler_CCI_V1/Ruler_CCI_V1.kicad_pcb (KiCad board)
At the start: 2 copper layers, 155 x 25 mm, 53 parts, among them Q1 BC107, Q2 BC107, Q3 BC107, Q4 BC107, Q5 BC107, SW1 SW_SPDT, U1 4017, U2 NE555D, U3 TPS61041DBV

Commit message: push panel
Parts:
- added 0201: R_0201_0603Metric, Resistor_SMD:R_0201_0603Metric, B.Cu at (63.2, 85.9)
- added 0402: R_0402_1005Metric, Resistor_SMD:R_0402_1005Metric, B.Cu at (61.1, 86.2)
- added 0603: R_0603_1608Metric, Resistor_SMD:R_0603_1608Metric, B.Cu at (58.6, 86.8)
- added 0805: R_0805_2012Metric, Resistor_SMD:R_0805_2012Metric, B.Cu at (55.7, 87.0)
- added 1206: R_1206_3216Metric, Resistor_SMD:R_1206_3216Metric, B.Cu at (52.4, 87.6)
- added 2010: R_2010_5025Metric, Resistor_SMD:R_2010_5025Metric, B.Cu at (48.4, 88.5)
- added BGA: BGA-121_9.0x9.0mm_Layout11x11_P0.8mm_Ball0.4mm_Pad0.35mm_NS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, Package_BGA:BGA-121_9.0x9.0mm_Layout11x11_P0.8mm_Ball0.4mm_Pad0.35mm_NSMD, B.Cu at (169.2, 88.8)
- added DEL SMT: LED_1206_3216Metric, LED_SMD:LED_1206_3216Metric, B.Cu at (48.5, 98.4)
- added M2: MountingHole_2.2mm_M2_DIN965_Pad, MountingHole:MountingHole_2.2mm_M2_DIN965_Pad, F.Cu at (194.5, 87.1)
- added M2,5: MountingHole_2.7mm_M2.5_DIN965_Pad, MountingHole:MountingHole_2.7mm_M2.5_DIN965_Pad, F.Cu at (194.5, 92.9)
- added M3: MountingHole_3.2mm_M3_DIN965_Pad, MountingHole:MountingHole_3.2mm_M3_DIN965_Pad, F.Cu at (194.5, 99.7)
- added QFP: LQFP-52_10x10mm_P0.65mm, Package_QFP:LQFP-52_10x10mm_P0.65mm, B.Cu at (157.0, 90.2)
- added REF**: TestPoint_Loop_D2.50mm_Drill1.0mm, TestPoint:TestPoint_Loop_D2.50mm_Drill1.0mm, F.Cu at (103.5, 99.4)
- added REF**: TestPoint_Pad_D4.0mm, TestPoint:TestPoint_Pad_D4.0mm, B.Cu at (100.9, 86.2)
- added REF**: TestPoint_Pad_1.5x1.5mm, TestPoint:TestPoint_Pad_1.5x1.5mm, B.Cu at (104.9, 94.6)
- added REF**: TestPoint_Pad_D3.0mm, TestPoint:TestPoint_Pad_D3.0mm, B.Cu at (101.4, 91.0)
- added REF**: TestPoint_Pad_1.0x1.0mm, TestPoint:TestPoint_Pad_1.0x1.0mm, B.Cu at (104.6, 97.2)
- added REF**: TestPoint_Pad_D1.0mm, TestPoint:TestPoint_Pad_D1.0mm, B.Cu at (102.4, 97.2)
- added REF**: OSHW-Symbol_13.4x12mm_SilkScreen, Symbol:OSHW-Symbol_13.4x12mm_SilkScreen, B.Cu at (181.5, 89.8)
- added REF**: TestPoint_Pad_4.0x4.0mm, TestPoint:TestPoint_Pad_4.0x4.0mm, B.Cu at (106.1, 86.2)
- added REF**: KiCad-Logo_8mm_SilkScreen, Symbol:KiCad-Logo_8mm_SilkScreen, B.Cu at (181.4, 100.8)
- added REF**: TestPoint_Pad_3.0x3.0mm, TestPoint:TestPoint_Pad_3.0x3.0mm, B.Cu at (105.6, 91.0)
- added REF**: TestPoint_Pad_D1.5mm, TestPoint:TestPoint_Pad_D1.5mm, B.Cu at (102.1, 94.6)
- added SOIC-16: SOIC-16_3.9x9.9mm_P1.27mm, Package_SO:SOIC-16_3.9x9.9mm_P1.27mm, B.Cu at (70.2, 96.8)
- added SOIC-4: SOIC-4_4.55x2.6mm_P1.27mm, Package_SO:SOIC-4_4.55x2.6mm_P1.27mm, B.Cu at (90.7, 93.2)
- added SOIC-8: SOIC-8_3.9x4.9mm_P1.27mm, Package_SO:SOIC-8_3.9x4.9mm_P1.27mm, B.Cu at (80.1, 94.3)
- added SOT-23: SOT-23, Package_TO_SOT_SMD:SOT-23, B.Cu at (70.2, 85.7)
- added SOT-323: SOT-323_SC-70, Package_TO_SOT_SMD:SOT-323_SC-70, B.Cu at (80.1, 85.7)
- added SOT-523: SOT-523, Package_TO_SOT_SMD:SOT-523, B.Cu at (90.6, 85.6)
Routing:
- net PWM: track 30.5 -> 47.9 mm
Other:
- board text added: "+"
- board text added: "-"
- board text added: "Anode"
- board text added: "Cathode"
- board text added: "Composantes passive SMT"
- board text added: "Définir les fonctionnalités voulues Recherche de composantes Création de schéma électrique Déverminage du schéma électrique (DRC) Association des symboles à leurs footprints Définir dimension du PCB Définir le stackup du PCB Placer les composantes Routage entre pièces (attention au courant) Nettoyage de la sérigraphie Déverminage du PCB (DRC) Envoie en production"
- board text added: "Schéma fait par: Miriam Caisse PCB fait par: Jacob Tucotte"
- board text added: "Small Outline Integrated Circuit (SOIC)"
- board text added: "Small Outline Transistor (SOT)"
- board text added: "To do list:"
- board text added: "Variété de points de test"
